Commit message: feat: fishbot working version，复制小鱼6.1开始的全部完整源码，ros2_control可正常工作，用于diff对比bug

File: src/fishbot_description/urdf/first_robot.urdf (robot description, URDF)
Before this commit: robot first_robot, 2 links, 1 joints
Joints:
- joint imu_joint: origin xyz=0.0 0.0 0.03 rpy=0.0 0.0 0.0 -> xyz=0 0 0.03 rpy=0 0 0

File: src/fishbot_description/urdf/first_robot.xacro (robot description, xacro)
@@ -1,48 +1,41 @@
 <?xml version="1.0"?>
 <robot xmlns:xacro="http://www.ros.org/wiki/xacro" name="first_robot">
-    <xacro:macro name='base_link' params = 'length radius'>
+    <!-- 声明 base 模块 -->
+    <xacro:macro name="base_link" params="length radius">
         <link name="base_link">
-        <!-- 部件的外观描述 -->
             <visual>
-                <!-- 沿着自己几何中心的偏移和旋转量 -->
-                <origin xyz="0.0 0.0 0.0" rpy="0.0 0.0 0.0"/>
-                <!-- 几何形状 -->
+                <origin xyz="0 0 0" rpy="0 0 0" />
                 <geometry>
-                    <!-- 圆柱体 radius 半径0.1m ;length 高度0.12m -->
-                    <cylinder radius="${radius}" length="${length}"/>
+                    <cylinder length="${length}" radius="${length}" />
                 </geometry>
-                <!-- 材质颜色描述 -->
-                <material name='white'>
-                    <color rgba="1.0 1.0 1.0 0.5"/>
+                <material name="blue">
+                    <color rgba="0.1 0.1 1.0 0.5" />
                 </material>
             </visual>
         </link>
     </xacro:macro>
-    <xacro:macro name='imu_link' params ='imu_name xyz'>
-         <!-- 机器人的IMU部件，惯性测量传感器 -->
+    <!-- 声明 IMU 模块 -->
+    <xacro:macro name="imu_link" params="imu_name xyz">
         <link name="${imu_name}_link">
-            <!-- 部件的外观描述 -->
             <visual>
-                <!-- 沿着自己几何中心的偏移和旋转量 -->
-                <origin xyz="0.0 0.0 0.0" rpy="0.0 0.0 0.0"/>
-                <!-- 几何形状 -->
+                <origin xyz="0 0 0" rpy="0 0 0" />
                 <geometry>
-                    <box size="0.02 0.02 0.02"/>
+                    <box size="0.02 0.02 0.02" />
                 </geometry>
-                <!-- 材质颜色描述 -->
-                <material name='black'>
-                    <color rgba="0.0 0.0 0.0 0.5"/>
-                </material>
             </visual>
+            <material name="black">
+                <color rgba="0 0 0 0.5" />
+            </material>
         </link>
-        <!-- 机器人的关节，用于组合机器人的部件 -->
         <joint name="${imu_name}_joint" type="fixed">
-            <parent link="base_link"/>
-            <child link="${imu_name}_link"/>
-            <origin xyz="${xyz}" rpy="0.0 0.0 0.0"/>
+            <parent link="base_link" />
+            <child link="${imu_name}_link" />
+            <origin xyz="${xyz}" />
         </joint>
     </xacro:macro>
-    <xacro:base_link length='0.12' radius='0.1'/>
-    <xacro:imu_link imu_name='imu_up' xyz='0.0 0.0 0.03'/>
-    <xacro:imu_link imu_name='imu_down' xyz='0.0 0.0 -0.03'/>
+    <!-- 传递参数调用 base_link 模块 -->
+    <xacro:base_link length="0.12" radius="0.1" />
+    <!-- 传递参数调用 imu 模块 -->
+    <xacro:imu_link imu_name="imu_up" xyz="0 0 0.02" />
+    <xacro:imu_link imu_name="imu_down" xyz="0 0 -0.02" />
 </robot>

File: src/fishbot_description/urdf/fishbot/actuator/caster.urdf.xacro (robot description, xacro)
@@ -1,48 +1,39 @@
 <?xml version="1.0"?>
 <robot xmlns:xacro="http://www.ros.org/wiki/xacro">
-<xacro:include filename="$(find fishbot_description)/urdf/fishbot/common_inertia.xacro"/>
-    <xacro:macro name='caster_xacro' params ='caster_name xyz'>
-         <!-- 机器人的IMU部件，惯性测量传感器 -->
-        <link name="${caster_name}_link">
-            <!-- 部件的外观描述 -->
+   <xacro:include filename="$(find fishbot_description)/urdf/fishbot/common_inertia.xacro" />
+    <xacro:macro name="caster_xacro" params="caster_name xyz">
+        <link name="${caster_name}_caster_link">
             <visual>
-                <!-- 沿着自己几何中心的偏移和旋转量 -->
-                <origin xyz="0.0 0.0 0.0" rpy="0 0.0 0.0"/>
-                <!-- 几何形状 -->
+                <origin xyz="0 0 0" rpy="0 0 0" />
                 <geometry>
-                    <sphere radius="0.016"/>
+                    <sphere radius="0.016" />
                 </geometry>
-                <!-- 材质颜色描述 -->
-                <material name='yellow'>
-                    <color rgba="1.0 1.0 0.0 0.8"/>
+                <material name="black">
+                    <color rgba="0.0 0.0 0.0 0.8"/>
                 </material>
             </visual>
             <collision>
-                <!-- 沿着自己几何中心的偏移和旋转量 -->
-                <origin xyz="0.0 0.0 0.0" rpy="0 0.0 0.0"/>
-                <!-- 几何形状 -->
+                <origin xyz="0 0 0" rpy="0 0 0" />
                 <geometry>
-                    <sphere radius="0.016"/>
+                    <sphere radius="0.016" />
                 </geometry>
-                <!-- 材质颜色描述 -->
-                <material name='yellow'>
-                    <color rgba="1.0 1.0 0.0 0.8"/>
+                <material name="black">
+                    <color rgba="0.0 0.0 0.0 0.8"/>
                 </material>
             </collision>
-            <xacro:sphere_inertia m='0.05' r='0.016' />
+            <xacro:sphere_inertia m="0.01" r="0.016" />
         </link>
-        <!-- 机器人的关节，用于组合机器人的部件 -->
-        <joint name="${caster_name}_joint" type="fixed">
-            <parent link="base_link"/>
-            <child link="${caster_name}_link"/>
-            <origin xyz="${xyz}"/>
+        <gazebo reference="${caster_name}_caster_link">
+            <mu1 value="0.0" />
+            <mu2 value="0.0" />
+            <kp value="1000000000.0" />
+            <kd value="1.0" />
+        </gazebo>
+        <joint name="${caster_name}_caster_joint" type="fixed">
+            <parent link="base_link" />
+            <child link="${caster_name}_caster_link" />
+            <origin xyz="${xyz}" />
+            <axis xyz="0 0 0" />
         </joint>
-        <gazebo reference='${caster_name}_link'>
-            <mu1 value='0.0'/>  #切向摩擦系数
-            <mu2 value='0.0'/>  #法向摩擦系数
-            <kp value='1000000000.0'/>  #接触刚度系数
-            <kd value='1.0'/>  #阻尼系数
-            <material>Gazebo/Yellow</material>
-        </gazebo>
     </xacro:macro>
 </robot>

File: src/fishbot_description/urdf/fishbot/actuator/wheel.urdf.xacro (robot description, xacro)
@@ -1,49 +1,39 @@
 <?xml version="1.0"?>
 <robot xmlns:xacro="http://www.ros.org/wiki/xacro">
-<xacro:include filename="$(find fishbot_description)/urdf/fishbot/common_inertia.xacro"/>
-    <xacro:macro name='wheel_xacro' params ='wheel_name xyz'>
-         <!-- 机器人的IMU部件，惯性测量传感器 -->
-        <link name="${wheel_name}_link">
-            <!-- 部件的外观描述 -->
+   <xacro:include filename="$(find fishbot_description)/urdf/fishbot/common_inertia.xacro" />
+    <xacro:macro name="wheel_xacro" params="wheel_name xyz">
+        <link name="${wheel_name}_wheel_link">
             <visual>
-                <!-- 沿着自己几何中心的偏移和旋转量 -->
-                <origin xyz="0.0 0.0 0.0" rpy="1.57079 0.0 0.0"/>
-                <!-- 几何形状 -->
+                <origin xyz="0 0 0" rpy="1.57079 0 0" />
                 <geometry>
-                    <cylinder radius="0.032" length="0.04"/>
+                    <cylinder length="0.04" radius="0.032" />
                 </geometry>
-                <!-- 材质颜色描述 -->
-                <material name='yellow'>
-                    <color rgba="1.0 1.0 0.0 0.8"/>
+                <material name="black">
+                    <color rgba="0.0 0.0 0.0 0.8"/>
                 </material>
             </visual>
             <collision>
-                <!-- 沿着自己几何中心的偏移和旋转量 -->
-                <origin xyz="0.0 0.0 0.0" rpy="1.57079 0.0 0.0"/>
-                <!-- 几何形状 -->
+                <origin xyz="0 0 0" rpy="1.57079 0 0" />
                 <geometry>
-                    <cylinder radius="0.032" length="0.04"/>
+                    <cylinder length="0.04" radius="0.032" />
                 </geometry>
-                <!-- 材质颜色描述 -->
-                <material name='yellow'>
-                    <color rgba="1.0 1.0 0.0 0.8"/>
+                <material name="black">
+                    <color rgba="0.0 0.0 0.0 0.8"/>
                 </material>
             </collision>
-            <xacro:cylinder_inertia m='0.05' r='0.032' h = '0.04' />
+            <xacro:cylinder_inertia m="0.1" h="0.04" r="0.032"/>
         </link>
-        <!-- 机器人的关节，用于组合机器人的部件 -->
-        <joint name="${wheel_name}_joint" type="continuous">
-            <parent link="base_link"/>
-            <child link="${wheel_name}_link"/>
-            <origin xyz="${xyz}"/>
-            <axis xyz="0.0 1.0 0.0"/>
+        <gazebo reference="${wheel_name}_wheel_link">
+            <mu1 value="20.0" />
+            <mu2 value="20.0" />
+            <kp value="1000000000.0" />
+            <kd value="1.0" />
+        </gazebo>
+        <joint name="${wheel_name}_wheel_joint" type="continuous">
+            <parent link="base_link" />
+            <child link="${wheel_name}_wheel_link" />
+            <origin xyz="${xyz}" />
+            <axis xyz="0 1 0" />
         </joint>
-        <gazebo reference='${wheel_name}_link'>
-            <mu1 value='20.0'/>  #切向摩擦系数
-            <mu2 value='20.0'/>  #法向摩擦系数
-            <kp value='1000000000.0'/>  #接触刚度系数
-            <kd value='1.0'/>  #阻尼系数
-            <material>Gazebo/Yellow</material>
-        </gazebo>
     </xacro:macro>
 </robot>

File: src/fishbot_description/urdf/fishbot/base.urdf.xacro (robot description, xacro)
@@ -1,43 +1,33 @@
 <?xml version="1.0"?>
 <robot xmlns:xacro="http://www.ros.org/wiki/xacro">
-    <xacro:include filename="$(find fishbot_description)/urdf/fishbot/common_inertia.xacro"/>
-    <xacro:macro name='base_xacro' params = 'length radius'>
-        <!-- 虚拟部件,不存在实体 -->
-        <link name="base_footprint" />
+   <xacro:include filename="$(find fishbot_description)/urdf/fishbot/common_inertia.xacro" />
+    <xacro:macro name="base_xacro" params="length radius">
+     <link name="base_footprint" />
+        <joint name="base_joint" type="fixed">
+            <parent link="base_footprint" />
+            <child link="base_link" />
+            <origin xyz="0.0 0.0 ${length/2.0+0.032-0.001}" rpy="0 0 0" />
+        </joint>
         <link name="base_link">
-        <!-- 部件的外观描述 -->
             <visual>
-                <!-- 沿着自己几何中心的偏移和旋转量 -->
-                <origin xyz="0.0 0.0 0.0" rpy="0.0 0.0 0.0"/>
-                <!-- 几何形状 -->
+                <origin xyz="0 0 0.0" rpy="0 0 0" />
                 <geometry>
-                    <!-- 圆柱体 radius 半径0.1m ;length 高度0.12m -->
-                    <cylinder radius="${radius}" length="${length}"/>
+                    <cylinder length="${length}" radius="${length}" />
                 </geometry>
-                <!-- 材质颜色描述 -->
-                <material name='white'>
-                    <color rgba="1.0 1.0 1.0 0.5"/>
+                <material name="blue">
+                    <color rgba="0.1 0.1 1.0 0.5"/>
                 </material>
             </visual>
             <collision>
-                <!-- 沿着自己几何中心的偏移和旋转量 -->
-                <origin xyz="0.0 0.0 0.0" rpy="0.0 0.0 0.0"/>
-                <!-- 几何形状 -->
+                <origin xyz="0 0 0.0" rpy="0 0 0" />
                 <geometry>
-                    <!-- 圆柱体 radius 半径0.1m ;length 高度0.12m -->
-                    <cylinder radius="${radius}" length="${length}"/>
+                    <cylinder length="${length}" radius="${length}" />
                 </geometry>
-                <!-- 材质颜色描述 -->
-                <material name='white'>
-                    <color rgba="1.0 1.0 1.0 0.5"/>
+                <material name="blue">
+                    <color rgba="0.1 0.1 1.0 0.5"/>
                 </material>
             </collision>
-            <xacro:cylinder_inertia m='1.0' r='${radius}' h='${length}' />
+            <xacro:cylinder_inertia m="1.0" r="${radius}" h="${length}"/>
         </link>
-        <joint name="joint_name" type="fixed">
-            <origin xyz="0.0 0.0 ${length/2.0 + 0.032 - 0.001}" rpy="0.0 0.0 0.0"/>
-            <parent link="base_footprint"/>
-            <child link="base_link"/>
-        </joint>
     </xacro:macro>
 </robot>

File: src/fishbot_description/urdf/fishbot/plugins/gazebo_control_plugin.xacro (robot description, xacro)
@@ -1,5 +1,5 @@
 <?xml version="1.0"?>
-<robot xmlns:xacro="http://www.ros.org/wiki/xacro" >
-    <xacro:macro name = 'gazebo_control_plugin'>
+<robot xmlns:xacro="http://www.ros.org/wiki/xacro">
+    <xacro:macro name="gazebo_control_plugin">
         <gazebo>
             <plugin name='diff_drive' filename='libgazebo_ros_diff_drive.so'>
@@ -13,8 +13,8 @@
                 <left_joint>left_wheel_joint</left_joint>
                 <right_joint>right_wheel_joint</right_joint>
-                <!-- kinematics 运动学设置，控制机器人角速度线速度时需要知道轮子之间的距离和轮子的半径 -->
+                <!-- kinematics -->
                 <wheel_separation>0.2</wheel_separation>
                 <wheel_diameter>0.064</wheel_diameter>
-                <!-- limits 轮子的限制 -->
+                <!-- limits -->
                 <max_wheel_torque>20</max_wheel_torque>
                 <max_wheel_acceleration>1.0</max_wheel_acceleration>
@@ -27,4 +27,4 @@
             </plugin>
         </gazebo>
-    </xacro:macro>
+   </xacro:macro>
 </robot>

File: src/fishbot_description/urdf/fishbot/plugins/gazebo_sensor_plugin.xacro (robot description, xacro)
@@ -1,8 +1,8 @@
 <?xml version="1.0"?>
-<robot xmlns:xacro="http://www.ros.org/wiki/xacro" >
-    <xacro:macro name = 'gazebo_sensor_plugin'>
-        <gazebo reference = 'laser_link'>
-            <sensor name = 'laserscan' type = 'ray'>
-                <plugin name='laserscan' filename='libgazebo_ros_ray_sensor.so'>
+<robot xmlns:xacro="http://www.ros.org/wiki/xacro">
+    <xacro:macro name="gazebo_sensor_plugin">
+        <gazebo reference="laser_link">
+            <sensor name="laserscan" type="ray">
+                <plugin name="laserscan" filename="libgazebo_ros_ray_sensor.so">
                     <ros>
                         <namespace>/</namespace>
@@ -16,7 +16,7 @@
                 <update_rate>5</update_rate>
                 <pose>0 0 0 0 0 0</pose>
-                <!-- 激光传感器配置 -->
+								<!-- 激光传感器配置 -->
                 <ray>
-                    <!-- 扫描范围设置 -->
+                    <!-- 设置扫描范围 -->
                     <scan>
                         <horizontal>
@@ -27,5 +27,5 @@
                         </horizontal>
                     </scan>
-                    <!-- 设置扫描范围 -->
+                    <!-- 设置扫描距离 -->
                     <range>
                         <min>0.120000</min>
@@ -40,101 +40,99 @@
                     </noise>
                 </ray>
-             </sensor>
-        </gazebo>
-        <!--imu设置  -->
-        <gazebo reference="imu_link">
-            <sensor name="imu_sensor" type="imu">
-                <plugin name="imu_plugin" filename="libgazebo_ros_imu_sensor.so">
-                    <ros>
-                        <namespace>/</namespace>
-                        <remapping>~/out:=imu</remapping>
-                    </ros>
-                    <initial_orientation_as_reference>false</initial_orientation_as_reference>
-                </plugin>
-                <update_rate>100</update_rate>
-                <always_on>true</always_on>
-                <!-- 六轴噪声设置 -->
-                <imu>
-                    <angular_velocity>
-                        <x>
-                            <noise type="gaussian">
-                                <mean>0.0</mean>
-                                <stddev>2e-4</stddev>
-                                <bias_mean>0.0000075</bias_mean>
-                                <bias_stddev>0.0000008</bias_stddev>
-                            </noise>
-                        </x>
-                        <y>
-                            <noise type="gaussian">
-                                <mean>0.0</mean>
-                                <stddev>2e-4</stddev>
-                                <bias_mean>0.0000075</bias_mean>
-                                <bias_stddev>0.0000008</bias_stddev>
-                            </noise>
-                        </y>
-                        <z>
-                            <noise type="gaussian">
-                                <mean>0.0</mean>
-                                <stddev>2e-4</stddev>
-                                <bias_mean>0.0000075</bias_mean>
-                                <bias_stddev>0.0000008</bias_stddev>
-                            </noise>
-                        </z>
-                    </angular_velocity>
-                    <linear_acceleration>
-                        <x>
-                            <noise type="gaussian">
-                                <mean>0.0</mean>
-                                <stddev>1.7e-2</stddev>
-                                <bias_mean>0.1</bias_mean>
-                                <bias_stddev>0.001</bias_stddev>
-                            </noise>
-                        </x>
-                        <y>
-                            <noise type="gaussian">
-                                <mean>0.0</mean>
-                                <stddev>1.7e-2</stddev>
-                                <bias_mean>0.1</bias_mean>
-                                <bias_stddev>0.001</bias_stddev>
-                            </noise>
-                        </y>
-                        <z>
-                            <noise type="gaussian">
-                                <mean>0.0</mean>
-                                <stddev>1.7e-2</stddev>
-                                <bias_mean>0.1</bias_mean>
-                                <bias_stddev>0.001</bias_stddev>
-                            </noise>
-                        </z>
-                    </linear_acceleration>
-                </imu>
             </sensor>
         </gazebo>
-        <!-- 相机camera设置 -->
-        <gazebo reference="camera_link">
-            <sensor type="depth" name="camera_sensor">
-                <plugin name="depth_camera" filename="libgazebo_ros_camera.so">
-                    <frame_name>camera_optical_link</frame_name>
-                </plugin>
-                <always_on>true</always_on>
-                <update_rate>10</update_rate>
-                <camera name="camera">
-                    <horizontal_fov>1.5009831567</horizontal_fov>
-                    <image>
-                        <width>800</width>
-                        <height>600</height>
-                        <format>R8G8B8</format>
-                    </image>
-                    <distortion>
-                        <k1>0.0</k1>
-                        <k2>0.0</k2>
-                        <k3>0.0</k3>
-                        <p1>0.0</p1>
-                        <p2>0.0</p2>
-                        <center>0.5 0.5</center>
-                    </distortion>
-                </camera>
-            </sensor>
-        </gazebo>
+<gazebo reference="imu_link">
+    <sensor name="imu_sensor" type="imu">
+        <plugin name="imu_plugin" filename="libgazebo_ros_imu_sensor.so">
+            <ros>
+                <namespace>/</namespace>
+                <remapping>~/out:=imu</remapping>
+            </ros>
+            <initial_orientation_as_reference>false</initial_orientation_as_reference>
+        </plugin>
+        <update_rate>100</update_rate>
+        <always_on>true</always_on>
+        <!-- 六轴噪声设置 -->
+        <imu>
+            <angular_velocity>
+                <x>
+                    <noise type="gaussian">
+                        <mean>0.0</mean>
+                        <stddev>2e-4</stddev>
+                        <bias_mean>0.0000075</bias_mean>
+                        <bias_stddev>0.0000008</bias_stddev>
+                    </noise>
+                </x>
+                <y>
+                    <noise type="gaussian">
+                        <mean>0.0</mean>
+                        <stddev>2e-4</stddev>
+                        <bias_mean>0.0000075</bias_mean>
+                        <bias_stddev>0.0000008</bias_stddev>
+                    </noise>
+                </y>
+                <z>
+                    <noise type="gaussian">
+                        <mean>0.0</mean>
+                        <stddev>2e-4</stddev>
+                        <bias_mean>0.0000075</bias_mean>
+                        <bias_stddev>0.0000008</bias_stddev>
+                    </noise>
+                </z>
+            </angular_velocity>
+            <linear_acceleration>
+                <x>
+                    <noise type="gaussian">
+                        <mean>0.0</mean>
+                        <stddev>1.7e-2</stddev>
+                        <bias_mean>0.1</bias_mean>
+                        <bias_stddev>0.001</bias_stddev>
+                    </noise>
+                </x>
+                <y>
+                    <noise type="gaussian">
+                        <mean>0.0</mean>
+                        <stddev>1.7e-2</stddev>
+                        <bias_mean>0.1</bias_mean>
+                        <bias_stddev>0.001</bias_stddev>
+                    </noise>
+                </y>
+                <z>
+                    <noise type="gaussian">
+                        <mean>0.0</mean>
+                        <stddev>1.7e-2</stddev>
+                        <bias_mean>0.1</bias_mean>
+                        <bias_stddev>0.001</bias_stddev>
+                    </noise>
+                </z>
+            </linear_acceleration>
+        </imu>
+    </sensor>
+</gazebo>
     </xacro:macro>
+<gazebo reference="camera_link">
+    <sensor type="depth" name="camera_sensor">
+        <plugin name="depth_camera" filename="libgazebo_ros_camera.so">
+            <frame_name>camera_optical_link</frame_name>
+        </plugin>
+        <always_on>true</always_on>
+        <update_rate>10</update_rate>
+        <camera name="camera">
+            <horizontal_fov>1.5009831567</horizontal_fov>
+            <image>
+                <width>800</width>
+                <height>600</height>
+                <format>R8G8B8</format>
+            </image>
+            <distortion>
+                <k1>0.0</k1>
+                <k2>0.0</k2>
+                <k3>0.0</k3>
+                <p1>0.0</p1>
+                <p2>0.0</p2>
+                <center>0.5 0.5</center>
+            </distortion>
+        </camera>
+    </sensor>
+</gazebo>
 </robot>
