Commit message: feat: fishbot working version，复制小鱼6.1开始的全部完整源码，ros2_control可正常工作，用于diff对比bug

File: src/fishbot_description/urdf/fishbot/sensor/camera.urdf.xacro (robot description, xacro)
@@ -1,50 +1,39 @@
 <?xml version="1.0"?>
 <robot xmlns:xacro="http://www.ros.org/wiki/xacro">
-<xacro:include filename="$(find fishbot_description)/urdf/fishbot/common_inertia.xacro"/>
-    <xacro:macro name='camera_xacro' params ='xyz'>
-         <!-- 机器人的camera部件 -->
+   <xacro:include filename="$(find fishbot_description)/urdf/fishbot/common_inertia.xacro" />
+    <xacro:macro name="camera_xacro" params="xyz">
+        <!-- ============相机模块================ -->
         <link name="camera_link">
-            <!-- 部件的外观描述 -->
             <visual>
-                <!-- 沿着自己几何中心的偏移和旋转量 -->
-                <origin xyz="0.0 0.0 0.0" rpy="0.0 0.0 0.0"/>
-                <!-- 几何形状 -->
+                <origin xyz="0 0 0.0" rpy="0 0 0" />
                 <geometry>
-                    <box size="0.02 0.10 0.02"/>
+                    <box size="0.02 0.10 0.02" />
                 </geometry>
-                <!-- 材质颜色描述 -->
-                <material name='green'>
-                    <color rgba="0.0 1.0 0.0 0.8"/>
+                <material name="black">
+                    <color rgba="0.0 0.0 0.0 0.8"/>
                 </material>
             </visual>
             <collision>
-                <!-- 沿着自己几何中心的偏移和旋转量 -->
-                <origin xyz="0.0 0.0 0.0" rpy="0.0 0.0 0.0"/>
-                <!-- 几何形状 -->
+                <origin xyz="0 0 0.0" rpy="0 0 0" />
                 <geometry>
-                    <box size="0.02 0.10 0.02"/>
+                    <box size="0.02 0.10 0.02" />
                 </geometry>
-                <!-- 材质颜色描述 -->
-                <material name='green'>
-                    <color rgba="0.0 1.0 0.0 0.8"/>
+                <material name="black">
+                    <color rgba="0.0 0.0 0.0 0.8"/>
                 </material>
             </collision>
-            <xacro:box_inertia m='0.1' w = '0.02' h = '0.10' d = '0.02' />
+            <xacro:box_inertia m="0.01" w="0.02" h="0.10" d="0.02" />
         </link>
         <link name="camera_optical_link"></link>
-        <!-- 机器人的关节，用于组合机器人的部件 -->
+        <joint name="camera_optical_joint" type="fixed">
+            <parent link="camera_link" />
+            <child link="camera_optical_link" />
+            <origin xyz="0 0 0" rpy="${-pi/2} 0 ${-pi/2}" />
+        </joint>
         <joint name="camera_joint" type="fixed">
-            <parent link="base_link"/>
-            <child link="camera_link"/>
-            <origin xyz="${xyz}" rpy = '0.0 0.0 0.0' />
+            <parent link="base_link" />
+            <child link="camera_link" />
+            <origin xyz="${xyz}" />
         </joint>
-        <joint name="camera_optical_joint" type="fixed">
-            <parent link="camera_link"/>
-            <child link="camera_optical_link"/>
-            <origin xyz="0 0 0" rpy = '${-pi/2} 0.0 ${-pi/2}' />
-        </joint>
-        <gazebo reference='camera_link'>
-            <material>Gazebo/Green</material>
-        </gazebo>
     </xacro:macro>
 </robot>

File: src/fishbot_description/urdf/fishbot/sensor/imu.urdf.xacro (robot description, xacro)
@@ -1,44 +1,32 @@
 <?xml version="1.0"?>
 <robot xmlns:xacro="http://www.ros.org/wiki/xacro">
-<xacro:include filename="$(find fishbot_description)/urdf/fishbot/common_inertia.xacro"/>
-    <xacro:macro name='imu_xacro' params ='xyz'>
-         <!-- 机器人的IMU部件，惯性测量传感器 -->
+   <xacro:include filename="$(find fishbot_description)/urdf/fishbot/common_inertia.xacro" />
+    <xacro:macro name="imu_xacro" params="xyz">
         <link name="imu_link">
-            <!-- 部件的外观描述 -->
             <visual>
-                <!-- 沿着自己几何中心的偏移和旋转量 -->
-                <origin xyz="0.0 0.0 0.0" rpy="0.0 0.0 0.0"/>
-                <!-- 几何形状 -->
+                <origin xyz="0 0 00" rpy="0 0 0" />
                 <geometry>
-                    <box size="0.02 0.02 0.02"/>
+                    <box size="0.02 0.02 0.02" />
                 </geometry>
-                <!-- 材质颜色描述 -->
-                <material name='black'>
-                    <color rgba="0.0 0.0 0.0 0.8"/>
+                <material name="black">
+                    <color rgba="0 0 0 0.8" />
                 </material>
             </visual>
             <collision>
-                <!-- 沿着自己几何中心的偏移和旋转量 -->
-                <origin xyz="0.0 0.0 0.0" rpy="0.0 0.0 0.0"/>
-                <!-- 几何形状 -->
+                <origin xyz="0 0 00" rpy="0 0 0" />
                 <geometry>
-                    <box size="0.02 0.02 0.02"/>
+                    <box size="0.02 0.02 0.02" />
                 </geometry>
-                <!-- 材质颜色描述 -->
-                <material name='black'>
-                    <color rgba="0.0 0.0 0.0 0.8"/>
+                <material name="black">
+                    <color rgba="0 0 0 0.8" />
                 </material>
             </collision>
-            <xacro:box_inertia m='0.05' w = '0.02' h = '0.02' d = '0.02' />
+            <xacro:box_inertia m="0.01" w="0.02" d="0.02" h="0.02"/>
         </link>
-        <!-- 机器人的关节，用于组合机器人的部件 -->
         <joint name="imu_joint" type="fixed">
-            <parent link="base_link"/>
-            <child link="imu_link"/>
-            <origin xyz="${xyz}"/>
+            <parent link="base_link" />
+            <child link="imu_link" />
+            <origin xyz="${xyz}" />
         </joint>
-        <gazebo reference='imu_link'>
-            <material>Gazebo/Red</material>
-        </gazebo>
     </xacro:macro>
 </robot>

File: src/fishbot_description/urdf/fishbot/sensor/laser.urdf.xacro (robot description, xacro)
@@ -1,81 +1,66 @@
 <?xml version="1.0"?>
 <robot xmlns:xacro="http://www.ros.org/wiki/xacro">
-<xacro:include filename="$(find fishbot_description)/urdf/fishbot/common_inertia.xacro"/>
-    <xacro:macro name='laser_xacro' params ='xyz'>
-         <!-- 机器人的laser部件,雷达支撑杆 -->
+   <xacro:include filename="$(find fishbot_description)/urdf/fishbot/common_inertia.xacro" />
+    <xacro:macro name="laser_xacro" params="xyz">
+        <gazebo reference="laser_cylinder_link">
+            <material>Gazebo/Black</material>
+        </gazebo>
+        <gazebo reference="laser_link">
+            <material>Gazebo/Black</material>
+        </gazebo>
+        <!-- ============雷达支撑杆================ -->
         <link name="laser_cylinder_link">
-            <!-- 部件的外观描述 -->
             <visual>
-                <!-- 沿着自己几何中心的偏移和旋转量 -->
-                <origin xyz="0.0 0.0 0.0" rpy="0.0 0.0 0.0"/>
-                <!-- 几何形状 -->
+                <origin xyz="0 0 0" rpy="0 0 0" />
                 <geometry>
-                    <cylinder radius="0.01" length="0.10"/>
+                    <cylinder length="0.10" radius="0.01" />
                 </geometry>
-                <!-- 材质颜色描述 -->
-                <material name='green'>
-                    <color rgba="0.0 1.0 0.0 0.8"/>
+                <material name="black">
+                    <color rgba="0.0 0.0 0.0 0.8" />
                 </material>
             </visual>
             <collision>
-                <!-- 沿着自己几何中心的偏移和旋转量 -->
-                <origin xyz="0.0 0.0 0.0" rpy="0.0 0.0 0.0"/>
-                <!-- 几何形状 -->
+                <origin xyz="0 0 0" rpy="0 0 0" />
                 <geometry>
-                    <cylinder radius="0.01" length="0.10"/>
+                    <cylinder length="0.10" radius="0.01" />
                 </geometry>
-                <!-- 材质颜色描述 -->
-                <material name='green'>
-                    <color rgba="0.0 1.0 0.0 0.8"/>
+                <material name="black">
+                    <color rgba="0.0 0.0 0.0 0.8" />
                 </material>
             </collision>
-            <xacro:cylinder_inertia m='0.05' r='0.01' h='0.10' />
+            <xacro:cylinder_inertia m="0.01" r="0.01" h="0.10" />
         </link>
-         <!-- 机器人的laser部件,雷达主体 -->
+        <joint name="laser_cylinder_joint" type="fixed">
+            <parent link="base_link" />
+            <child link="laser_cylinder_link" />
+            <origin xyz="${xyz}" />
+        </joint>
+        <!-- ============雷达================ -->
         <link name="laser_link">
-            <!-- 部件的外观描述 -->
             <visual>
-                <!-- 沿着自己几何中心的偏移和旋转量 -->
-                <origin xyz="0.0 0.0 0.0" rpy="0.0 0.0 0.0"/>
-                <!-- 几何形状 -->
+                <origin xyz="0 0 0" rpy="0 0 0" />
                 <geometry>
-                    <cylinder radius="0.02" length="0.02"/>
+                    <cylinder length="0.02" radius="0.02" />
                 </geometry>
-                <!-- 材质颜色描述 -->
-                <material name='green'>
-                    <color rgba="0.0 1.0 0.0 0.8"/>
+                <material name="black">
+                    <color rgba="0.0 0.0 0.0 0.8" />
                 </material>
             </visual>
             <collision>
-                <!-- 沿着自己几何中心的偏移和旋转量 -->
-                <origin xyz="0.0 0.0 0.0" rpy="0.0 0.0 0.0"/>
-                <!-- 几何形状 -->
+                <origin xyz="0 0 0" rpy="0 0 0" />
                 <geometry>
-                    <cylinder radius="0.02" length="0.02"/>
+                    <cylinder length="0.02" radius="0.02" />
                 </geometry>
-                <!-- 材质颜色描述 -->
-                <material name='green'>
-                    <color rgba="0.0 1.0 0.0 0.8"/>
+                <material name="black">
+                    <color rgba="0.0 0.0 0.0 0.8" />
                 </material>
             </collision>
-            <xacro:cylinder_inertia m='0.10' r='0.02' h='0.02' />
+            <xacro:cylinder_inertia m="0.03" r="0.02" h="0.02" />
         </link>
-        <!-- 机器人的关节，用于组合机器人的部件 -->
         <joint name="laser_joint" type="fixed">
-            <parent link="laser_cylinder_link"/>
-            <child link="laser_link"/>
-            <origin xyz="0.0 0.0 0.05"/>
+            <parent link="laser_cylinder_link" />
+            <child link="laser_link" />
+            <origin xyz="0 0 0.05" />
         </joint>
-        <joint name="laser_cylinder_joint" type="fixed">
-            <parent link="base_link"/>
-            <child link="laser_cylinder_link"/>
-            <origin xyz="${xyz}"/>
-        </joint>
-        <gazebo reference='laser_cylinder_link'>
-            <material>Gazebo/Green</material>
-        </gazebo>
-        <gazebo reference='laser_link'>
-            <material>Gazebo/Green</material>
-        </gazebo>
     </xacro:macro>
 </robot>
